File: electronics/Bugsy/Bugsy.kicad_sch (KiCad schematic)
At the start: 16 parts, among them J1 Raspberry_Pi_2_3, J2 Conn_01x08, J3 Conn_02x26_Odd_Even, J4 Conn_01x08, J5 Conn_01x08_Socket, J6 Conn_01x08_Pin, M1 Motor_DC, M2 Motor_DC, SW1 SW_DPST_x2, U1 ESP32-WROOM-32, U2 L298N, U3 MPU6050, U4 CH340C, U5 LCD-016N002L

Commit message: upgrading electronics and writing docs
Parts:
- added BT2: Battery, symbol Device:Battery
- added U6: TMU3-0511, Converter_DCDC:Converter_DCDC_TRACO_TMU3-05xx_12xx_THT, symbol Converter_DCDC:TMU3-0511
Connections:
- net +24V: now also SW1.1 (A), U2.4 (Vs), U6.2 (+Vin); no longer BT1.1 (+)
- net +5V: now also U1.2 (VDD), U2.9 (Vss), U6.4 (+Vout)
- net GND: now also U2.8 (GND), BT2.2 (-), U6.1 (-Vin), U6.3 (-Vout); no longer SW1.2 (B)
- net +12V: now reaches BT1.2 (-)
- net +12V: now also BT2.1 (+); no longer SW1.1 (A)
- net UART_RX: now reaches U1.30 (IO18)
- net UART_TX: now reaches U1.31 (IO19)
- net PWM_MR_F: now reaches U2.10 (IN3)
- net PWM_MR_B: now reaches U2.12 (IN4)
- net PWM_ML_F: now reaches U2.5 (IN1)
- net PWM_ML_B: now reaches U2.7 (IN2)
- new net: BT1.1 (+), SW1.2 (B)
- no-connect marks 11 -> 21
Other:
- note added: "11.1V rated"
- note added: "3 cell lipo"
- note added: "Left motor"
- note added: "Onboard LED"
- note added: "Right motor"
- note removed: "22.2V rated"
- note removed: "6 cell Lipo"
- moved on the sheet: BT1, SW1A, U1

Commit message: massive code improvements
Parts:
- removed J3: Conn_02x26_Odd_Even, symbol Connector_Generic:Conn_02x26_Odd_Even
- added A1.R1: 22k, symbol Device:R
- added A1.R2: 1k, symbol Device:R
- added BZ1: Buzzer, symbol Device:Buzzer
- added D1: LED_ARGB, symbol Device:LED_ARGB
- added J1: Conn_02x16_Odd_Even, symbol Connector_Generic:Conn_02x16_Odd_Even
- added J20: Conn_01x05_Pin, symbol Connector:Conn_01x05_Pin
- added J6: Conn_01x05_Socket, symbol Connector:Conn_01x05_Socket
- added J8: Conn_01x03_Pin, symbol Connector:Conn_01x03_Pin
- added M2.J1: USB_B_Micro, symbol Connector:USB_B_Micro
- added M2.U2: CH340C, Package_SO:SOIC-16_3.9x9.9mm_P1.27mm, symbol Interface_USB:CH340C
- added M3.J1: USB_B, symbol Connector:USB_B
- added R3, R4, R5: R, symbol Device:R
- added SW20: RotaryEncoder_Switch, symbol Device:RotaryEncoder_Switch
- added U1: SX1276, Package_DFN_QFN:QFN-28-1EP_6x6mm_P0.65mm_EP4.8x4.8mm, symbol RF:SX1276
- added U3: PCA9685PW, Package_SO:TSSOP-28_4.4x9.7mm_P0.65mm, symbol Driver_LED:PCA9685PW
- added U7: DHT11, Sensor:Aosong_DHT11_5.5x12.0_P2.54mm, symbol Sensor:DHT11
- M3.U1: renamed from A1; value Arduino_UNO_R2 -> Arduino
- renumbered BT1 to A1.BT1, BT2 to A1.BT2, SW1 to A1.SW1, U6 to A1.U1, U1 to A2.U1, J6 to J10, U3 to M, U4 to M3.U2, J1 to U120
Connections:
- net +24V: now also A1.R1.1
- net +5V: now also M3.U2.16 (VCC), U120.2 (5V), U120.4 (5V), J1.1 (Pin_1), J1.2 (Pin_2), M2.J1.1 (VBUS), M2.U2.16 (VCC), M3.J1.1 (VBUS), U3.28 (VDD)
- net GND: now also A2.U1.1 (GND), A2.U1.15 (GND), A2.U1.38 (GND), A2.U1.39 (GND), M3.U2.1 (GND), U120.14 (GND), U120.20 (GND), U120.25 (GND), U120.30 (GND), U120.34 (GND), U120.39 (GND), U120.6 (GND), U120.9 (GND), A1.R2.2, J1.31 (Pin_31), J1.32 (Pin_32), J20.5 (Pin_5), M2.J1.5 (GND), M2.J1.6 (Shield), M2.U2.1 (GND), M3.J1.4 (GND), M3.J1.5 (Shield), R3.2, R4.2, R5.2, U3.1 (A0), U3.14 (VSS), U3.2 (A1), U3.24 (A5), U3.3 (A2), U3.4 (A3), U3.5 (A4)
- net PWM_ML_B: now also A2.U1.10 (IO25)
- net PWM_ML_F: now also A2.U1.37 (IO23)
- net PWM_MR_B: now also A2.U1.12 (IO27)
- net PWM_MR_F: now also A2.U1.11 (IO26)
- net at M3.U2.2 (TXD): now also M3.U1.15 (D0/RX)
- net at M3.U2.3 (RXD): now also M3.U1.16 (D1/TX)
- net at M3.U2.5 (UD+): now also M3.J1.3 (D+)
- net at M3.U2.6 (UD-): now also M3.J1.2 (D-)
- net I2C_SDA: now reaches A2.U1.33 (IO21)
- net at A2.U1.34 (RXD0/IO3): now also M2.U2.3 (RXD)
- net at A2.U1.35 (TXD0/IO1): now also M2.U2.2 (TXD)
- net I2C_SCL: now reaches A2.U1.36 (IO22)
- net BATTERY_MEAS: now reaches A2.U1.6 (IO34)
- net BATTERY_MEAS: now also A1.R1.2, A1.R2.1
- net RASP_UART3_RX: now reaches U120.29 (GCLK1/GPIO5)
- net RASP_UART3_TX: now reaches U120.7 (GCLK0/GPIO4)
- net UART_CORE_TRADER_RX: no longer names the net of J2.2 (Pin_2)
- net UART_CORE_TRADER_TX: no longer names the net of J2.1 (Pin_1)
- net UART_RPI_TRADER_RX: no longer names the net of J2.4 (Pin_4)
- net UART_RPI_TRADER_TX: no longer names the net of J2.3 (Pin_3)
- new net: J8.1 (Pin_1), U7.1 (VDD)
- new net: J8.2 (Pin_2), U7.2 (DATA)
- new net: J8.3 (Pin_3), U7.4 (GND)
- new net: U1.15 (GND), U1.23 (GND), U1.26 (GND), U1.29 (GND)
- new net: M2.J1.3 (D+), M2.U2.5 (UD+)
- new net: M2.J1.2 (D-), M2.U2.6 (UD-)
- new net CK: J20.3 (Pin_3), R4.1, SW20.B
- new net DT: J20.2 (Pin_2), R3.1, SW20.A
- new net EXT_PWM_1: U3.6 (LED0)
- new net EXT_PWM_2: U3.7 (LED1)
- new net SW: J20.4 (Pin_4), R5.1, SW20.S2
- new net VCC: J20.1 (Pin_1), SW20.C, SW20.S1
- no-connect marks 21 -> 34
Other:
- note added: "A1 - Power supply"
- note added: "A2 - NodeMCU32S"
- note added: "DHT11 - Temperature & Humidity"
- note added: "M3 - Arduino Mega2560"
- note added: "M3.U3"
- note added: "Rotary Encoder module"
- note added: "U20"
- note added: "U30"
- note added: "UART0"
- note added: "UART3"
- note added: "Voltage devider to scale down battery - 2.5dB ADC -> 0-1.5V range on ESP32 - Max ~26V when fully charged, scaling down by 22 / 1 gives ~1.2V max"
- note removed: "Onboard LED"
- moved on the sheet: A1.U1, A2.U1, J10, J2, J4, J5, M, M1, M2, M3.U1, M3.U2, U120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
